File: trap-pcb.sch (KiCad schematic (older format))
At the start: 77 parts, among them J1 Conn_01x15, J2 Conn_01x15, M1 Motor_DC, Q1 Q_NMOS_GSD, Q2 Q_NMOS_GSD, Q3 Q_NMOS_GSD, Q4 Q_NMOS_GSD, Q5 Q_NMOS_GSD, Q6 Q_NMOS_GSD, Q7 Q_NMOS_GSD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

Commit message: Fix lcsc part number
Parts:
- C27: JLCPCB SMD C134765 -> C14663
Changed lines of the file:
@@
 F 2 "Capacitor_SMD:C_0603_1608Metric" H 8938 3450 50  0001 C CNN
 F 3 "~" H 8900 3600 50  0001 C CNN
-F 4 "C134765" H 8900 3600 50  0001 C CNN "JLCPCB SMD"
+F 4 "C14663" H 8900 3600 50  0001 C CNN "JLCPCB SMD"
 	1    8900 3600
 	1    0    0    -1
